Commit message: Add files via upload

File: src/thepotbot/description/robot_core.xacro (robot description, xacro)
@@ -98,8 +98,8 @@
     <joint name="laser_joint" type="fixed">
         <parent link="chassis"/>
-        <child link="laser_frame"/>
+        <child link="base_laser"/>
         <origin xyz="0 0 ${ratio*(chassis_height+1.00)/2}" rpy="0 0 0"/>
     </joint>
-    <link name="laser_frame">
+    <link name="base_laser">
         <visual>
             <geometry>
@@ -123,12 +123,13 @@
         </visual>
     </link>
+<!--
     <joint name="valve_joint" type="revolute">
         <parent link="valve_frame"/>
-        <child link="valve"/>
+        <child link="valve_front"/>
         <origin xyz="0 0 ${ratio*(chassis_length/2+0.25)}" rpy="0 ${pi/2} 0"/>
         <axis xyz="-1 0.0 0.0"/>
         <limit lower="0.0" upper="${pi/2}" effort="100" velocity="100"/>
     </joint>
-    <link name="valve">
+    <link name="valve_front">
         <visual>
             <geometry>
@@ -138,3 +139,4 @@
         </visual>
     </link>
+-->
 </robot>

Commit message: Add files via upload

File: src/thepotbot/description/robot_core.xacro (robot description, xacro)
@@ -25,4 +25,12 @@
     <!-- BASE LINK -->
     <link name="base_link">
+    </link>
+    <!-- BASE_FOOTPRINT LINK -->
+    <joint name="base_footprint_joint" type="fixed">
+        <parent link="base_link"/>
+        <child link="base_footprint"/>
+        <origin xyz="0 0 0" rpy="0 0 0"/>
+    </joint>
+    <link name="base_footprint">
     </link>
     <!-- CHASSIS LINK -->
